File: Design/Smart_Plant_patch.sch (EAGLE design)
At the start: 67 parts, among them IC1 AMS1117-3.3, IC2 TLC555CDR, IC3 AHT20, IC4 TP4056, J2 USBC-6P, Q1 IRLML0100, Q2 ALS-PT19-315C, T1 MMBT2222A, T2 LBSS84LT1G, U1 ESP-32S

Commit message: Released designs from V1R1 with the patch board
Parts:
- removed C10, C16: 10uF, rcl:C-USC0603
- removed C11, C6: 100nF, rcl:C-USC0603
- removed C12: 22uF, rcl:C-USC0603
- removed C13, C14, C17, C18, C19, C25, C27, C28, C7, C9: 1uF, rcl:C-USC0603
- removed C15: 0.1uF, rcl:C-USC0603
- removed C2, C26: 4.7uF, rcl:C-USC0603
- removed C3: 0.47nF, rcl:C-USC0603
- removed C5: 10nF, rcl:C-USC0603
- removed D1, D2, D3: SS14, SparkFun-DiscreteSemi:DIODE-SCHOTTKY-SS14
- removed D4: LL4148, SpaceDIY_semiconductors:LL4148
- removed FPC: E-PAPER-FPC, SpaceDIY_connectors:E-PAPER-FPC
- removed IC1: AMS1117-3.3, SparkFun-IC-Power:V_REG_LD1117VXXLD1117-SMD
- removed IC2: TLC555CDR, linear:NE555D
- removed IC3: AHT20, SamacSys_Parts:AHT20
- removed J2: USBC-6P, SpaceDIY_connectors:USBC-6P
- removed J4: (no value), SparkFun-Connectors:CONN_02-JST-2-PTH-NO_SILK
- removed J5: (no value), SparkFun-Connectors:CONN_04PTH
- removed L3: 10uH, microbuilder:INDUCTORNR401
- removed Q1: IRLML0100, Parts:IRLML2060TRPBF
- removed Q2: ALS-PT19-315C, SparkFun-DiscreteSemi:PHOTOTRANSISTORPT17-21C-L41-TR8
- removed R1, R10, R12, R14, R15, R16, R7: 10k, rcl:R-US_R0603
- removed R11: 1k, rcl:R-US_R0603
- removed R13: 0.47, rcl:R-US_R0603
- removed R17: 220, rcl:R-US_R0603
- removed R18: 240k, rcl:R-US_R0603
- removed R19, R8: 1M, rcl:R-US_R0603
- removed R2: 330R, rcl:R-US_R0603
- removed R3: 1.5k, rcl:R-US_R0603
- removed R9: 10K, rcl:R-US_R0603
- removed S1: Flash, SpaceDIY_electromechanical:MOMENTARY-SWITCH-SPST-SMD-5.2MM-TALL
- removed S2: Reset, SpaceDIY_electromechanical:MOMENTARY-SWITCH-SPST-SMD-5.2MM-TALL
- removed T1: MMBT2222A, JLC PCB Basic Parts_loc:T_NPN_MMBT2222A-1P_CHANGJ_SOT23-BEC
- removed T2: LBSS84LT1G, JLC PCB Basic Parts_loc:T_P-MOSFET_LBSS84LT1G_LRC_SOT23-GSD
- removed TP1, TP2: TPB1,27, testpad:TPB1,27
- removed U1: ESP-32S, esp32:ESP-32S
- added C23: 10uF, rcl:C-USC0603
- added IC6: RT9080-33GJ5, SamacSys_Parts:RT9080-33GJ5
- added J6: USB-C-POWER, SpaceDIY_connectors:USB-C-POWER
- added J8: (no value), SpaceDIY_connectors:CONN_02-JST-2MM-SMT
- renumbered C1 to C21, C4 to C20, C8 to C22, IC4 to IC5, J1 to J3, LED1 to LED3, LED2 to LED4, R4 to R20, R5 to R21, R6 to R22
Connections:
- removed net BATTERY: R18.1, R19.2, U1.IO35
- removed net BUSY: FPC.9, U1.IO25
- removed net DC: FPC.11, U1.IO27
- removed net DISPCS: FPC.12, U1.IO15
- removed net GDR: FPC.2, Q1.G, R1.1
- removed net IO0: R12.2, S1.2, U1.IO0
- removed net LIGHT: Q2.E, R14.1, U1.IO33
- removed net MOISTURE: C7.1, D4.C, R8.1, U1.IO32
- removed net MOSI: FPC.14, U1.IO14
- removed net N$10: C15.1, C16.1, IC3.VDD, R17.2
- removed net N$11: C9.2, FPC.5
- removed net N$12: C13.2, FPC.18
- removed net N$13: C14.2, FPC.20
- removed net N$14: C17.2, FPC.22
- removed net N$15: C18.2, FPC.24
- removed net N$16: C26.2, D2.A, D3.C
- removed net N$17: C26.1, D1.A, L3.1, Q1.D
- removed net N$18: R11.2, T1.B
- removed net N$31: C27.2, FPC.4
- removed net N$32: C28.2, FPC.19
- removed net N$5: C3.1, IC2.THR, IC2.TR, R3.2
- removed net N$7: IC2.DIS, R2.2, R3.1
- removed net N$8: C5.2, IC2.CV
- removed net N$9: R10.2, T1.C, T2.G
- removed net OUT: IC2.Q, R7.2, TP1.TP
- removed net PROBE: D4.A, R7.1
- removed net RESE: FPC.3, Q1.S, R13.1
- removed net RESET: FPC.10, U1.IO26
- removed net RST: R9.1, S2.2, U1.EN
- removed net RX: J5.4, U1.U0RXD
- removed net SCL: IC3.SCL, R15.2, U1.IO22
- removed net SCLK: FPC.13, U1.IO13
- removed net SDA: IC3.SDA, R16.2, U1.IO21
- removed net SENS: R11.1, U1.IO16
- removed net TX: J5.3, U1.U0TXD
- removed net VGH: C19.1, D1.C, FPC.21
- removed net VGL: C25.1, D3.A, FPC.23
- removed net VSENS: C6.1, IC2.R, IC2.V+, Q2.C, R15.1, R16.1, R17.1, R2.1, T2.D, TP2.TP
- net 3.3V: now also C23.1, IC6.VOUT; no longer C10.1, C11.1, C12.1, C2.1, FPC.15, FPC.16, IC1.OUT, J5.1, L3.2, R10.1, R12.1, R9.2, T2.S, U1.3V3
- net GND: now also C23.2, IC5.TEMP, IC6.GND, J6.GND, J8.1; no longer C10.2, C11.2, C12.2, C13.1, C14.1, C15.2, C16.2, C17.1, C18.1, C19.2, C2.2, C25.2, C27.1, C28.1, C3.2, C5.1, C6.2, C7.2, C9.1, D2.C, FPC.17, FPC.8, IC1.GND, IC2.GND, IC3.GND, IC5.CE, J2.GND, J4.1, J5.2, R1.2, R13.2, R14.2, R18.2, R8.2, S1.1, S2.1, T1.E, U1.GND@1, U1.GND@2, U1.GND@3, U1.GND@4
- net VBAT: now also IC6.EN, IC6.VIN, J8.2; no longer IC1.IN, J4.2, R19.1
- net VIN: now also IC5.CE, J6.VBUS; no longer IC5.TEMP, J2.VBUS
Other:
- note removed: "Battery monitoring"
- note removed: "Capacitive moisture sensor"
- note removed: "High switch for power supply"
- note removed: "Light sensor"
- note removed: "Microcontroller"
- note removed: "Reset & Flash switches"
- note removed: "Serial port"
- note removed: "Temperature & humidity sensor"
- note removed: "eInk Display"
