File: Design/Smart_Plant.sch (EAGLE design)
At the start: 95 parts, among them IC1 TP4056, IC2 TLC555CDR, IC3 AHT20, IC4 RT9080-33GJ5, IC5 LC709203F/MH, IC6 VEML7700-TR, J6 USB-C, Q1 IRLML0100, T1 MMBT2222A, T2 LBSS84LT1G, U2 ESP32-WROOM-32, X5 ESP32-S3QFN54, Y2 40MHz

Commit message: Design V1R3
Parts:
- removed C21: 5.6pF, esp32-thing-temp:5.6PF-50V-5%(0603)
- removed C46, C48, C55, C57, C62, C63: 1uF, microbuilder:CAP_CERAMIC_0402NO
- removed C47, C52, C53, C54, C56, C58: 0.1uF, microbuilder:CAP_CERAMIC_0402NO
- removed C49: 22uF, microbuilder:CAP_CERAMIC0805-NOOUTLINE
- removed C59, C60: 16pF, microbuilder:CAP_CERAMIC_0402NO
- removed C61: 1uF, SpaceDIY_passive_components:C0402
- removed E2: ANTENNA, esp32-thing-temp:ANTENNATRACE-TUNED
- removed IC5: LC709203F/MH, adafruit_sensor:LC709203F/MH
- removed J4: (no value), SpaceDIY_connectors:CONN_02-JST-2MM-SMT
- removed L2: 2.7nH, SparkFun-Passives:INDUCTOR0603
- removed L5: 2nH, microbuilder:RESISTOR_0402NO
- removed R29: 0, microbuilder:RESISTOR_0402NO
- removed R30: 1Meg, microbuilder:RESISTOR_0402NO
- removed R31: 10K, SpaceDIY_passive_components:R0402
- removed U2: ESP32-WROOM-32, ESP32-WROOM-32:ESP32-WROOM-32
- removed X5: ESP32-S3QFN54, adafruit_wireless:ESP32-S3QFN54
- removed Y2: 40MHz, microbuilder:CRYSTAL_2X1.6MM
- added C12: 0.1uF, rcl:C-USC0603
- added IC7: MAX17048G+T10, SpaceDIY_IC:MAX17048G+T10
- added R36, R37: 5.1k, rcl:R-US_R0603
- added R9: 10K, rcl:R-US_R0603
- added U1: ESP32-S3-MINI-1-N8, SpaceDIY_modules:ESP32-S3-MINI-1-N8
- C20: value 2.4pF -> 10uF; device esp32-thing-temp:2.4PF-0603-50V-5% -> rcl:C-USC0603
- C40: value 1uF -> 0.1uF
- IC1: LCSC (none) -> C16581
- J1: device SparkFun-Connectors:CONN_02 -> SpaceDIY_connectors:BAT_CONN-JST-2MM-SMT
- J6: LCSC (none) -> C2765186
- LED1: LCSC (none) -> C2286
- LED2: LCSC (none) -> C72043
Connections:
- removed net !RESET: C61.1, R31.2, S2.2, X5.CHIP_PU
- removed net A2: X5.IO9
- removed net A3: X5.IO8
- removed net IO10_DBLTAP: C62.1, R30.2, X5.IO10
- removed net LIGHT: U2.IO33
- removed net LNA_IN1: C21.1, L2.1, X5.LNA_IN
- removed net MISO: X5.IO37
- removed net N$53: C59.1, X5.XTAL_P, Y2.2
- removed net N$54: C60.1, R29.1, Y2.1
- removed net N$55: R29.2, X5.XTAL_N
- removed net NEOPIX: X5.MTCK
- removed net NEOPIX_PWR: X5.IO38
- removed net SCK: X5.IO36
- removed net SCL1: X5.MTD0
- removed net SDA1: X5.MTDI
- removed net TRACE_ANT1: C20.1, C21.2, E2.SIGNAL
- removed net VDD3P3: C47.1, L5.2, X5.VDD3P3@0, X5.VDD3P3@1
- removed net VDD_SPI: C54.1, C55.1, X5.VDD_SPI
- new net +SOL: D6.A, R20.1
- new net N$35: J6.CC2, R36.2
- net 3.3V: now also C12.1, C20.1, R9.2, U1.3V3; no longer C46.1, C48.1, C49.1, C52.1, C53.1, C56.1, C57.1, C58.1, C63.1, L5.1, R31.1, U2.3V3, X5.IO21, X5.VDD3P3_CPU, X5.VDD3P3_RTC, X5.VDDA@0, X5.VDDA@1
- net BATTERY: now also U1.IO17; no longer U2.IO35, X5.IO18
- net BUSY: now also U1.IO33; no longer U2.IO25
- net D+: now also U1.IO20; no longer X5.IO20
- net D-: now also U1.IO19; no longer X5.IO19
- net DC: now also U1.IO37; no longer U2.IO27
- net DISPCS: now also U1.IO34; no longer U2.IO15
- net GND: now also C12.2, IC7.CTG, IC7.GND, IC7.QSTRT, J1.-, R36.1, R37.1, U1.GND; no longer C46.2, C47.2, C48.2, C49.2, C52.2, C53.2, C54.2, C55.2, C56.2, C57.2, C58.2, C59.2, C60.2, C61.2, C62.2, C63.2, E2.GND, IC5.TEST, IC5.VSS, J1.2, J4.1, L2.2, R30.1, U2.GND, X5.GND
- net IO0: now also U1.IO0; no longer U2.IO0, X5.IO0
- net MOISTURE: now also U1.IO15; no longer U2.IO32, X5.IO17
- net MOSI: now also U1.IO35; no longer U2.IO14, X5.IO35
- net N$46: now also J6.CC1, R37.2; no longer D6.A, J1.1, R20.1
- net RESET: now also U1.IO38; no longer U2.IO26
- net RST: now also R9.1, S2.2, U1.EN; no longer U2.EN
- net RX: now also U1.RXD0; no longer U2.RXD0, X5.U0RXD
- net SCL: now also IC7.SCL, U1.IO4; no longer IC5.SCL, U2.IO22, X5.IO6
- net SCLK: now also U1.IO36; no longer U2.IO13
- net SDA: now also IC7.SDA, U1.IO3; no longer IC5.SDA, U2.IO21, X5.IO7
- net SENS: now also U1.IO21; no longer U2.IO16, X5.IO4
- net TX: now also U1.TXD0; no longer U2.TXD0, X5.U0TXD
- net VBAT: now also IC7.CELL, IC7.VDD, J1.+; no longer IC5.VDD, J4.2
- net VSOLAR: now also U1.IO16; no longer U2.IO34
Other:
- note added: "Reset & Flash switches"

Commit message: First draft of the V2R1 design
Parts:
- removed U1: ESP32-S3-MINI-1-N8, SpaceDIY_modules:ESP32-S3-MINI-1-N8
- added IC5: ESP32-S2-MINI-1-N4R2, SpaceDIY_modules:ESP32-S2-MINI-1-N4R2
- IC6: device SpaceDIY_sensors:LIGHT_SENSOR -> SpaceDIY_sensors:LIGHT_SENSOR-TR
Connections:
- net 3.3V: now also IC5.3V3; no longer U1.3V3
- net BATTERY: now also IC5.IO2; no longer U1.IO17
- net BUSY: now also IC5.IO14; no longer U1.IO33
- net D+: now also IC5.IO20; no longer U1.IO20
- net D-: now also IC5.IO19; no longer U1.IO19
- net DC: now also IC5.IO13; no longer U1.IO37
- net DISPCS: now also IC5.IO10; no longer U1.IO34
- net GND: now also IC5.GND_1, IC5.GND_10, IC5.GND_11, IC5.GND_12, IC5.GND_13, IC5.GND_14, IC5.GND_15, IC5.GND_16, IC5.GND_17, IC5.GND_18, IC5.GND_19, IC5.GND_2, IC5.GND_20, IC5.GND_21, IC5.GND_22, IC5.GND_23, IC5.GND_24, IC5.GND_25, IC5.GND_26, IC5.GND_27, IC5.GND_28, IC5.GND_29, IC5.GND_3, IC5.GND_30, IC5.GND_31, IC5.GND_32, IC5.GND_33, IC5.GND_4, IC5.GND_5, IC5.GND_6, IC5.GND_7, IC5.GND_8, IC5.GND_9; no longer U1.GND
- net IO0: now also IC5.IO0; no longer U1.IO0
- net MOISTURE: now also IC5.IO1; no longer U1.IO15
- net MOSI: now also IC5.IO11; no longer U1.IO35
- net RESET: now also IC5.IO15; no longer U1.IO38
- net RST: now also IC5.EN; no longer U1.EN
- net RX: now also IC5.RXD0; no longer U1.RXD0
- net SCL: now also IC5.IO34; no longer U1.IO4
- net SCLK: now also IC5.IO12; no longer U1.IO36
- net SDA: now also IC5.IO33; no longer U1.IO3
- net SENS: now also IC5.IO4; no longer U1.IO21
- net TX: now also IC5.TXD0; no longer U1.TXD0
- net VSOLAR: now also IC5.IO3; no longer U1.IO16
Other:
- moved on the sheet: C12, C20, D6, IC6, R20, R21
